File: hw/ucode.sch (KiCad schematic (older format))
At the start: 13 parts

Commit message: working on device read/write signals
We will need to use the inverted outputs from the '175
flip flops latching the microcode signals in order to
ensure that the device-specific read/write signals are
high on reset.  This means using positive logic for
decoding the device ids.  NOR gates do the trick for
the GP registers, and the '238 decoder does the other
devices (it produces active high outputs, rather than
active low like the '138 decoder.)
Parts:
- removed U? (x6): 74LS00, symbol 74LS00
- added U? (x6): 74LS02, symbol 74LS02
- U? (x2): value 74LS138 -> 74LS238
Connections:
- net labels added: rdARHi, rdARLo, rdGPHi, rdGPLo, rdMem, rdPCHi, rdPCLo, wrARHi, wrARLo, wrGPHi, wrGPLo, wrMem, wrPCHi, wrPCLo
- net labels removed: -gpReadHi, -gpReadLo, -gpWriteHi, -gpWriteLo, -rdARHi, -rdARLo, -rdMem, -rdPCHi, -rdPCLo, -wrARHi, -wrARLo, -wrMem, -wrPCHi, -wrPCLo, VCC
- wire segments 125 -> 119
Other:
- note added: "Device read/write signals"
- note added: "Note: these are '238\ndecoders with active\nhigh outputs, not '138\ndecoders with active\nlow outputs"
- note added: "TODO: add '175 registers,\nuse inverted outputs as\ncleaned up ucode signals\n(from the device r/w\ngeneration EPROM)"
- moved on the sheet: U?
