File: hw/earlyrst.sch (KiCad schematic (older format))
At the start: 8 parts

Commit message: adding component references
Parts:
- gave numbers to parts that had none: 4
Connections:
- net lateRST: now reaches U203.11 (~Q2)

Commit message: added ucode output registers
Parts:
- U201: value 74LS393 -> 74HC393
- U202: value 74LS32 -> 74HC32
- U203: value 74LS175 -> 74HC175
- U204: value 74LS541 -> 74HC541
Changed lines of the file:
@@
 P 6600 4800
 F 0 "U204" H 6600 5375 50  0000 C BNN
-F 1 "74LS541" H 6600 4225 50  0000 C TNN
+F 1 "74HC541" H 6600 4225 50  0000 C TNN
 F 2 "" H 6600 4800 50  0001 C CNN
 F 3 "" H 6600 4800 50  0001 C CNN
@@
 P 3800 1900
 F 0 "U201" H 3950 2150 50  0000 C CNN
-F 1 "74LS393" H 4000 1650 50  0000 C CNN
+F 1 "74HC393" H 4000 1650 50  0000 C CNN
 F 2 "" H 3800 1900 50  0000 C CNN
 F 3 "" H 3800 1900 50  0000 C CNN
@@
 P 3800 2650
 F 0 "U201" H 3950 2900 50  0000 C CNN
-F 1 "74LS393" H 4000 2400 50  0000 C CNN
+F 1 "74HC393" H 4000 2400 50  0000 C CNN
 F 2 "" H 3800 2650 50  0000 C CNN
 F 3 "" H 3800 2650 50  0000 C CNN
@@
 P 8600 2300
 F 0 "U203" H 8600 2300 50  0000 C CNN
-F 1 "74LS175" H 8700 1900 50  0000 C CNN
+F 1 "74HC175" H 8700 1900 50  0000 C CNN
 F 2 "" H 8600 2300 50  0000 C CNN
 F 3 "" H 8600 2300 50  0000 C CNN
@@
 P 6450 1850
 F 0 "U202" H 6450 1900 50  0000 C CNN
-F 1 "74LS32" H 6450 1800 50  0000 C CNN
+F 1 "74HC32" H 6450 1800 50  0000 C CNN
 F 2 "" H 6450 1850 50  0000 C CNN
 F 3 "" H 6450 1850 50  0000 C CNN
@@
 P 6450 2300
 F 0 "U202" H 6450 2350 50  0000 C CNN
-F 1 "74LS32" H 6450 2250 50  0000 C CNN
+F 1 "74HC32" H 6450 2250 50  0000 C CNN
 F 2 "" H 6450 2300 50  0000 C CNN
 F 3 "" H 6450 2300 50  0000 C CNN
@@
 P 6450 2750
 F 0 "U202" H 6450 2800 50  0000 C CNN
-F 1 "74LS32" H 6450 2700 50  0000 C CNN
+F 1 "74HC32" H 6450 2700 50  0000 C CNN
 F 2 "" H 6450 2750 50  0000 C CNN
 F 3 "" H 6450 2750 50  0000 C CNN
@@
 P 2450 5200
 F 0 "U202" H 2450 5250 50  0000 C CNN
-F 1 "74LS32" H 2450 5150 50  0000 C CNN
+F 1 "74HC32" H 2450 5150 50  0000 C CNN
 F 2 "" H 2450 5200 50  0000 C CNN
 F 3 "" H 2450 5200 50  0000 C CNN
