File: hw/phase.sch (KiCad schematic (older format))
At the start: 9 parts

Commit message: adding component references
Parts:
- gave numbers to parts that had none: 3
Changed lines of the file:
@@
 CLK
 $Comp
-L 74LS175 U?
+L 74LS175 U303
 U 1 1 5929A5F9
 P 7000 3700
-F 0 "U?" H 7000 3700 50  0000 C CNN
+F 0 "U303" H 7000 3700 50  0000 C CNN
 F 1 "74LS175" H 7100 3300 50  0000 C CNN
 F 2 "" H 7000 3700 50  0001 C CNN
@@
 $EndComp
 $Comp
-L 74LS02 U?
+L 74LS02 U301
 U 1 1 5929A6F9
 P 3750 3150
-F 0 "U?" H 3750 3200 50  0000 C CNN
+F 0 "U301" H 3750 3200 50  0000 C CNN
 F 1 "74LS02" H 3800 3100 50  0000 C CNN
 F 2 "" H 3750 3150 50  0001 C CNN
@@
 $EndComp
 $Comp
-L 74LS02 U?
+L 74LS02 U301
 U 2 1 5929A716
 P 3750 3650
-F 0 "U?" H 3750 3700 50  0000 C CNN
+F 0 "U301" H 3750 3700 50  0000 C CNN
 F 1 "74LS02" H 3800 3600 50  0000 C CNN
 F 2 "" H 3750 3650 50  0001 C CNN
@@
 $EndComp
 $Comp
-L 74LS32 U?
+L 74LS32 U302
 U 1 1 5929AA34
 P 5250 3250
-F 0 "U?" H 5250 3300 50  0000 C CNN
+F 0 "U302" H 5250 3300 50  0000 C CNN
 F 1 "74LS32" H 5250 3200 50  0000 C CNN
 F 2 "" H 5250 3250 50  0001 C CNN
@@
 -opfetch
 $Comp
-L 74LS02 U?
+L 74LS02 U301
 U 3 1 5929B0A2
 P 3750 4800
-F 0 "U?" H 3750 4850 50  0000 C CNN
+F 0 "U301" H 3750 4850 50  0000 C CNN
 F 1 "74LS02" H 3800 4750 50  0000 C CNN
 F 2 "" H 3750 4800 50  0001 C CNN
@@
 $EndComp
 $Comp
-L 74LS02 U?
+L 74LS02 U301
 U 4 1 5929B12B
 P 3750 5300
-F 0 "U?" H 3750 5350 50  0000 C CNN
+F 0 "U301" H 3750 5350 50  0000 C CNN
 F 1 "74LS02" H 3800 5250 50  0000 C CNN
 F 2 "" H 3750 5300 50  0001 C CNN
@@
 $EndComp
 $Comp
-L 74LS32 U?
+L 74LS32 U302
 U 2 1 5929B25C
 P 5100 4900
-F 0 "U?" H 5100 4950 50  0000 C CNN
+F 0 "U302" H 5100 4950 50  0000 C CNN
 F 1 "74LS32" H 5100 4850 50  0000 C CNN
 F 2 "" H 5100 4900 50  0001 C CNN
@@
 	5900 4900 5700 4900
 $Comp
-L 74LS32 U?
+L 74LS32 U302
 U 3 1 5929BF66
 P 1650 6250
-F 0 "U?" H 1650 6300 50  0000 C CNN
+F 0 "U302" H 1650 6300 50  0000 C CNN
 F 1 "74LS32" H 1650 6200 50  0000 C CNN
 F 2 "" H 1650 6250 50  0001 C CNN
@@
 $EndComp
 $Comp
-L 74LS32 U?
+L 74LS32 U302
 U 4 1 5929C0A9
 P 1650 6700
-F 0 "U?" H 1650 6750 50  0000 C CNN
+F 0 "U302" H 1650 6750 50  0000 C CNN
 F 1 "74LS32" H 1650 6650 50  0000 C CNN
 F 2 "" H 1650 6700 50  0001 C CNN

Commit message: added ucode output registers
Parts:
- U301: value 74LS02 -> 74HC02
- U302: value 74LS32 -> 74HC32
- U303: value 74LS175 -> 74HC175
Changed lines of the file:
@@
 P 7000 3700
 F 0 "U303" H 7000 3700 50  0000 C CNN
-F 1 "74LS175" H 7100 3300 50  0000 C CNN
+F 1 "74HC175" H 7100 3300 50  0000 C CNN
 F 2 "" H 7000 3700 50  0001 C CNN
 F 3 "" H 7000 3700 50  0001 C CNN
@@
 P 3750 3150
 F 0 "U301" H 3750 3200 50  0000 C CNN
-F 1 "74LS02" H 3800 3100 50  0000 C CNN
+F 1 "74HC02" H 3800 3100 50  0000 C CNN
 F 2 "" H 3750 3150 50  0001 C CNN
 F 3 "" H 3750 3150 50  0001 C CNN
@@
 P 3750 3650
 F 0 "U301" H 3750 3700 50  0000 C CNN
-F 1 "74LS02" H 3800 3600 50  0000 C CNN
+F 1 "74HC02" H 3800 3600 50  0000 C CNN
 F 2 "" H 3750 3650 50  0001 C CNN
 F 3 "" H 3750 3650 50  0001 C CNN
@@
 P 5250 3250
 F 0 "U302" H 5250 3300 50  0000 C CNN
-F 1 "74LS32" H 5250 3200 50  0000 C CNN
+F 1 "74HC32" H 5250 3200 50  0000 C CNN
 F 2 "" H 5250 3250 50  0001 C CNN
 F 3 "" H 5250 3250 50  0001 C CNN
@@
 P 3750 4800
 F 0 "U301" H 3750 4850 50  0000 C CNN
-F 1 "74LS02" H 3800 4750 50  0000 C CNN
+F 1 "74HC02" H 3800 4750 50  0000 C CNN
 F 2 "" H 3750 4800 50  0001 C CNN
 F 3 "" H 3750 4800 50  0001 C CNN
@@
 P 3750 5300
 F 0 "U301" H 3750 5350 50  0000 C CNN
-F 1 "74LS02" H 3800 5250 50  0000 C CNN
+F 1 "74HC02" H 3800 5250 50  0000 C CNN
 F 2 "" H 3750 5300 50  0001 C CNN
 F 3 "" H 3750 5300 50  0001 C CNN
@@
 P 5100 4900
 F 0 "U302" H 5100 4950 50  0000 C CNN
-F 1 "74LS32" H 5100 4850 50  0000 C CNN
+F 1 "74HC32" H 5100 4850 50  0000 C CNN
 F 2 "" H 5100 4900 50  0001 C CNN
 F 3 "" H 5100 4900 50  0001 C CNN
@@
 P 1650 6250
 F 0 "U302" H 1650 6300 50  0000 C CNN
-F 1 "74LS32" H 1650 6200 50  0000 C CNN
+F 1 "74HC32" H 1650 6200 50  0000 C CNN
 F 2 "" H 1650 6250 50  0001 C CNN
 F 3 "" H 1650 6250 50  0001 C CNN
@@
 P 1650 6700
 F 0 "U302" H 1650 6750 50  0000 C CNN
-F 1 "74LS32" H 1650 6650 50  0000 C CNN
+F 1 "74HC32" H 1650 6650 50  0000 C CNN
 F 2 "" H 1650 6700 50  0001 C CNN
 F 3 "" H 1650 6700 50  0001 C CNN
