File: hw/pc.sch (KiCad schematic (older format))
At the start: 8 parts, among them U601 74HC191, U602 74HC191, U603 74HC191, U604 74HC191, U605 74HC10, U606 74HC08, U607 74HC541, U608 74HC541

Commit message: replace '193 with '393 in opfetch module
The '393 has two fewer pins, better use of breadboard space.
Changed lines of the file:
@@
 	9450 2850 9050 2850
 Wire Wire Line
-	9050 1500 9050 2850
-Wire Wire Line
-	1350 1500 9050 1500
+	9050 2850 9050 1500
+Wire Wire Line
+	9050 1500 1350 1500
 Wire Wire Line
 	7350 2850 6700 2850
@@
 	8400 3550 7550 3550
 Wire Wire Line
-	7550 3250 7550 3550
-Wire Wire Line
-	4300 3250 7550 3250
+	7550 3550 7550 3250
+Wire Wire Line
+	7550 3250 4300 3250
 Wire Wire Line
 	8900 2750 8900 3250
